Commit message: disable body collision shape

File: rsc/virtual_human.urdf (robot description, URDF)
Before this commit: robot amass_male, 20 links, 19 joints
Links:
- link chest: mass 8.0 -> 4.0; geometry visual sphere radius=0.07; visual sphere radius=0.07
- link lelbow: geometry collision box size=0.22 0.05 0.05; visual box size=0.22 0.04 0.04
- link lowerback: mass 5.0 -> 2.0; geometry visual sphere radius=0.065
- link lowerneck: geometry visual capsule length=0.0273 radius=0.030
- link upperback: mass 5.0 -> 2.0; geometry visual sphere length=0.125 radius=0.05
- link upperneck: geometry visual capsule length=0.035 radius=0.06

Commit message: fix collision shape

File: rsc/virtual_human.urdf (robot description, URDF)
Before this commit: robot amass_male, 20 links, 19 joints
Links:
- link lwrist: geometry collision box size=0.08 0.04 0.08; visual box size=0.08 0.04 0.08
- link rwrist: geometry collision box size=0.08 0.04 0.08; visual box size=0.08 0.04 0.08

Commit message: update virtual human with body collision

File: rsc/virtual_human.urdf (robot description, URDF)
Before this commit: robot amass_male, 20 links, 19 joints
Links:
- link chest: geometry collision sphere radius=0.07; collision sphere radius=0.07
- link lknee: geometry visual capsule length=0.325 radius=0.05
- link lowerback: geometry collision sphere radius=0.065; visual sphere radius=0.065
- link lowerneck: geometry collision capsule length=0.0273 radius=0.030; visual capsule length=0.0273 radius=0.030
- link rknee: geometry visual capsule length=0.325 radius=0.05
- link upperback: geometry collision sphere length=0.125 radius=0.05; visual sphere length=0.125 radius=0.05
- link upperneck: geometry collision capsule length=0.035 radius=0.06; visual capsule length=0.035 radius=0.06

Commit message: virtual human with wrist

File: rsc/virtual_human.urdf (robot description, URDF)
Before this commit: robot amass_male, 20 links, 19 joints
Joints:
- joint lwrist: axis 1 0 0 -> 0 0 1; limit (none) -> lower=-1.57 upper=1.57 effort=50.0 velocity=100.5; type fixed -> revolute
- joint rwrist: axis 1 0 0 -> 0 0 1; limit (none) -> lower=-1.57 upper=1.57 effort=50.0 velocity=100.5; type fixed -> revolute
